File: pcb/led-robot/led-robot.kicad_pcb (KiCad board)
At the start: 2 copper layers, 29.2 x 26.2 mm, 30 parts, among them J1 data, U1 MAX7219

Commit message: update
Other:
- board text added: "5V"
- board text added: "CLK"
- board text added: "DIN"
- board text added: "GND"
- board text added: "LOAD"
Changed lines of the file:
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@@
   (general
     (thickness 1.6)
-    (drawings 8)
+    (drawings 12)
     (tracks 247)
     (zones 0)
@@
     (tags "SOIC 1.27")
     (attr smd)
-    (fp_text reference U1 (at 0 8.8) (layer B.SilkS)
+    (fp_text reference U1 (at 0 -8.75) (layer B.SilkS)
       (effects (font (size 1 1) (thickness 0.15)) (justify mirror))
     )
@@
     (descr "Through hole straight pin header, 1x05, 2.54mm pitch, single row")
     (tags "Through hole pin header THT 1x05 2.54mm single row")
-    (fp_text reference J1 (at 0 2.33 90) (layer B.SilkS)
+    (fp_text reference J1 (at 0 2.75 180) (layer B.SilkS)
       (effects (font (size 1 1) (thickness 0.15)) (justify mirror))
     )
@@
     )
   )
+  (gr_text GND (at 193.25 94.25 270) (layer B.SilkS)
+    (effects (font (size 1.5 1.5) (thickness 0.3)) (justify mirror))
+  )
+  (gr_text 5V (at 190.5 95 270) (layer B.SilkS)
+    (effects (font (size 1.5 1.5) (thickness 0.3)) (justify mirror))
+  )
+  (gr_text DIN (at 188 94.5 270) (layer B.SilkS)
+    (effects (font (size 1.5 1.5) (thickness 0.3)) (justify mirror))
+  )
+  (gr_text CLK (at 185.25 94.5 270) (layer B.SilkS)
+    (effects (font (size 1.5 1.5) (thickness 0.3)) (justify mirror))
+  )
+  (gr_text LOAD (at 182.75 93.75 270) (layer B.SilkS)
+    (effects (font (size 1.5 1.5) (thickness 0.3)) (justify mirror))
+  )
   (gr_line (start 181 100.25) (end 181 100) (layer Edge.Cuts) (width 0.2))
   (gr_line (start 210.25 100.25) (end 181 100.25) (layer Edge.Cuts) (width 0.2))
@@
   (gr_line (start 181 81.75) (end 181 74) (layer Edge.Cuts) (width 0.2))
   (gr_line (start 181 100) (end 181 81.75) (layer Edge.Cuts) (width 0.2))
-  (gr_line (start 149.25 67.5) (end 219.25 67.5) (layer F.Fab) (width 0.2))
   (via (at 197 87) (size 0.8) (drill 0.4) (layers F.Cu B.Cu) (net 1))
   (segment (start 198.0625 88.0625) (end 197 87) (width 0.25) (layer F.Cu) (net 1))
