File: pcb/led-controller/led-controller.kicad_pcb (KiCad board)
At the start: 2 copper layers, 38 x 32 mm, 16 parts, among them J1 USB, J2 CP2102, J3 BUTTONS, J4 EYEs, J5 LEDs, J6 SRV, U1 ATmega328P-PU, Y1 16Mhz

Commit message: update final pcb
Routing:
- added copper zone on B.Cu, net GND
Changed lines of the file:
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@@
   (segment (start 182.88 68.252) (end 186.83499 72.20699) (width 0.25) (layer F.Cu) (net 28))
   (segment (start 182.88 66.802) (end 182.88 68.252) (width 0.25) (layer F.Cu) (net 28))
+  (zone (net 13) (net_name GND) (layer B.Cu) (hatch edge 0.508)
+    (connect_pads (clearance 0.508))
+    (min_thickness 0.254)
+    (fill yes (arc_segments 16) (thermal_gap 0.508) (thermal_bridge_width 0.508))
+    (polygon
+      (pts
+        (xy 192.8 58.2) (xy 179.8 58.2) (xy 179.8 55.2) (xy 168.2 55.2) (xy 168.2 58.2)
+        (xy 155.2 58.2) (xy 155.2 86.8) (xy 192.8 86.8) (xy 192.8 86.4)
+      )
+    )
+  )
 )
